File: Aurora.sch (KiCad schematic (older format))
At the start: 26 parts, among them J1 Conn_01x06_Female, J2 Barrel_Jack_Switch, Q1 BC547, Q2 J113, U1 TL072, U2 NE555P

Commit message: Correctly annotate output DC reference resistor and add to PCB
Parts:
- R9: renamed from R?; footprint (none) -> Resistor_THT:R_Axial_DIN0207_L6.3mm_D2.5mm_P2.54mm_Vertical
- renumbered R9 to R10, R10 to R11, R11 to R12
Changed lines of the file:
@@
 Connection ~ 7250 3500
 $Comp
-L Device:R R10
+L Device:R R11
 U 1 1 5F011CCA
 P 9200 3700
-F 0 "R10" V 9407 3700 50  0000 C CNN
+F 0 "R11" V 9407 3700 50  0000 C CNN
 F 1 "1k" V 9316 3700 50  0000 C CNN
 F 2 "Resistor_THT:R_Axial_DIN0207_L6.3mm_D2.5mm_P7.62mm_Horizontal" V 9130 3700 50  0001 C CNN
@@
 $EndComp
 $Comp
-L Device:R R9
+L Device:R R10
 U 1 1 5F011CD0
 P 9400 3400
-F 0 "R9" H 9470 3446 50  0000 L CNN
+F 0 "R10" H 9470 3446 50  0000 L CNN
 F 1 "47k" H 9470 3355 50  0000 L CNN
 F 2 "Resistor_THT:R_Axial_DIN0207_L6.3mm_D2.5mm_P7.62mm_Horizontal" V 9330 3400 50  0001 C CNN
@@
 	8550 3900 8600 3900
 $Comp
-L Device:R R11
+L Device:R R12
 U 1 1 5F011D01
 P 8800 3400
-F 0 "R11" H 8870 3446 50  0000 L CNN
+F 0 "R12" H 8870 3446 50  0000 L CNN
 F 1 "100" H 8870 3355 50  0000 L CNN
 F 2 "Resistor_THT:R_Axial_DIN0207_L6.3mm_D2.5mm_P7.62mm_Horizontal" V 8730 3400 50  0001 C CNN
@@
 Output
 $Comp
-L Device:R R?
+L Device:R R9
 U 1 1 5F0A905F
 P 5850 2800
-F 0 "R?" H 5920 2846 50  0000 L CNN
+F 0 "R9" H 5920 2846 50  0000 L CNN
 F 1 "1M" H 5920 2755 50  0000 L CNN
-F 2 "" V 5780 2800 50  0001 C CNN
+F 2 "Resistor_THT:R_Axial_DIN0207_L6.3mm_D2.5mm_P2.54mm_Vertical" V 5780 2800 50  0001 C CNN
 F 3 "~" H 5850 2800 50  0001 C CNN
 	1    5850 2800
@@
 	5850 2550 6000 2550
 $Comp
-L power:GND #PWR?
+L power:GND #PWR0101
 U 1 1 5F0ABEB5
 P 5850 3000
-F 0 "#PWR?" H 5850 2750 50  0001 C CNN
+F 0 "#PWR0101" H 5850 2750 50  0001 C CNN
 F 1 "GND" H 5855 2827 50  0000 C CNN
 F 2 "" H 5850 3000 50  0001 C CNN
