File: Aurora.kicad_pcb (KiCad board)
At the start: 2 copper layers, 54.6 x 52.7 mm, 30 parts, among them J1 Conn_01x06_Female, J2 Barrel_Jack_Switch, Q1 BC547, Q2 J113, U1 TL072, U2 TL074

Commit message: Correctly annotate output DC reference resistor and add to PCB
Parts:
- added R9: 1M, Resistor_THT:R_Axial_DIN0207_L6.3mm_D2.5mm_P2.54mm_Vertical, F.Cu at (113.0, 99.1)
- U2: value TL074 -> NE555P
- moved C6 1.91 mm to (114.2, 94.0)
- moved R1 1.27 mm to (118.1, 99.1)
- moved R8 1.27 mm to (109.2, 88.9), turned to 0 degrees
- renumbered R9 to R10, R10 to R11, R11 to R12
Routing:
- net Input: track 16.7 -> 21.0 mm
- net Output: track 8.71 -> 11.7 mm
- net +9VA: track 150.3 -> 149.6 mm
- net Net-(C6-Pad2): track 5.72 -> 5.08 mm

Commit message: Bump revision
Other:
- board text added: "NFX005 Aurora r03 Oct 2020 Steamed Hams!"
- board text removed: "NFX005 Aurora r02 Jul 2020 Steamed Hams!"
Changed lines of the file:
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@@
   (title_block
     (title Aurora)
-    (date 2020-07-11)
-    (rev r02)
+    (date 2020-10-04)
+    (rev r03)
     (company "Nuclear Lighthouse Studios")
     (comment 1 "CC BY-NC-SA")
@@
     )
   )
-  (gr_text "NFX005\nAurora r02\nJul 2020\nSteamed Hams!" (at 99.695 84.455) (layer F.SilkS)
+  (gr_text "NFX005\nAurora r03\nOct 2020\nSteamed Hams!" (at 99.695 84.455) (layer F.SilkS)
     (effects (font (size 1 1) (thickness 0.15)))
   )

Commit message: Properly connect trace between R1 and R2
Routing:
- net Net-(C3-Pad1): track 16.6 -> 17.9 mm
Other:
- board text added: "NFX005 Aurora r04 Jul 2021 Steamed Hams!"
- board text removed: "NFX005 Aurora r03 Oct 2020 Steamed Hams!"
Changed lines of the file:
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@@
-(kicad_pcb (version 20171130) (host pcbnew 5.1.6)
+(kicad_pcb (version 20171130) (host pcbnew 5.1.10)
   (general
     (thickness 1.6)
@@
   (title_block
     (title Aurora)
-    (date 2020-10-04)
-    (rev r03)
+    (date 2021-07-04)
+    (rev r04)
     (company "Nuclear Lighthouse Studios")
     (comment 1 "CC BY-NC-SA")
@@
     (add_net "Net-(C6-Pad2)")
     (add_net "Net-(C7-Pad1)")
-    (add_net "Net-(J1-Pad2)")
     (add_net "Net-(Q1-Pad1)")
     (add_net "Net-(Q1-Pad2)")
@@
     (add_net "Net-(R6-Pad2)")
     (add_net "Net-(R7-Pad1)")
-    (add_net "Net-(RV1-Pad3)")
-    (add_net "Net-(U2-Pad5)")
     (add_net Output)
   )
@@
     )
     (fp_text value 1M (at 1.27 2.37) (layer F.Fab)
-      (effects (font (size 1 1) (thickness 0.15)))
-    )
-    (fp_text user %R (at 1.27 -2.37) (layer F.Fab)
       (effects (font (size 1 1) (thickness 0.15)))
     )
@@
     (fp_line (start 3.59 1.5) (end 3.59 -1.5) (layer F.CrtYd) (width 0.05))
     (fp_line (start 3.59 -1.5) (end -1.5 -1.5) (layer F.CrtYd) (width 0.05))
+    (fp_text user %R (at 1.27 -2.37) (layer F.Fab)
+      (effects (font (size 1 1) (thickness 0.15)))
+    )
     (pad 2 thru_hole oval (at 2.54 0 180) (size 1.6 1.6) (drill 0.8) (layers *.Cu *.Mask)
       (net 1 GND))
@@
     )
   )
-  (gr_text "NFX005\nAurora r03\nOct 2020\nSteamed Hams!" (at 99.695 84.455) (layer F.SilkS)
+  (gr_text "NFX005\nAurora r04\nJul 2021\nSteamed Hams!" (at 99.695 84.455) (layer F.SilkS)
     (effects (font (size 1 1) (thickness 0.15)))
   )
@@
   (segment (start 130.694989 94.095011) (end 130.694989 90.285011) (width 0.5) (layer F.Cu) (net 5))
   (segment (start 120.65 99.06) (end 121.92 97.79) (width 0.5) (layer F.Cu) (net 5))
-  (segment (start 118.11 97.79) (end 118.11 93.98) (width 0.5) (layer F.Cu) (net 6))
   (segment (start 120.57 88.9) (end 121.92 88.9) (width 0.5) (layer F.Cu) (net 6))
   (segment (start 121.92 88.9) (end 125.73 92.71) (width 0.5) (layer F.Cu) (net 6))
@@
   (segment (start 118.11 93.98) (end 118.11 92.71) (width 0.5) (layer F.Cu) (net 6))
   (segment (start 118.11 92.71) (end 120.57 90.25) (width 0.5) (layer F.Cu) (net 6))
+  (segment (start 118.11 93.98) (end 118.11 99.06) (width 0.5) (layer F.Cu) (net 6))
   (segment (start 129.54 76.974998) (end 129.54 74.295) (width 0.5) (layer F.Cu) (net 7))
   (segment (start 131.225002 78.66) (end 129.54 76.974998) (width 0.5) (layer F.Cu) (net 7))
@@
   (segment (start 134.62 99.695) (end 138.43 95.885) (width 0.5) (layer F.Cu) (net 8))
   (segment (start 109.22 93.98) (end 109.22 88.9) (width 0.5) (layer F.Cu) (net 9))
-  (segment (start 107.315 72.39) (end 103.505 68.58) (width 0.5) (layer F.Cu) (net 19))
-  (segment (start 107.315 73.66) (end 107.315 72.39) (width 0.5) (layer F.Cu) (net 19))
-  (segment (start 93.98 64.135) (end 92.075 66.04) (width 0.5) (layer F.Cu) (net 19))
-  (segment (start 99.06 64.135) (end 93.98 64.135) (width 0.5) (layer F.Cu) (net 19))
-  (segment (start 103.505 68.58) (end 99.06 64.135) (width 0.5) (layer F.Cu) (net 19))
   (segment (start 92.075 72.39) (end 95.885 68.58) (width 0.5) (layer F.Cu) (net 10))
   (segment (start 92.075 73.66) (end 92.075 72.39) (width 0.5) (layer F.Cu) (net 10))
@@
   (segment (start 115.57 69.205499) (end 114.309501 67.945) (width 0.5) (layer F.Cu) (net 18))
   (segment (start 115.57 69.205499) (end 115.57 72.39) (width 0.5) (layer F.Cu) (net 18))
+  (segment (start 107.315 72.39) (end 103.505 68.58) (width 0.5) (layer F.Cu) (net 19))
+  (segment (start 107.315 73.66) (end 107.315 72.39) (width 0.5) (layer F.Cu) (net 19))
+  (segment (start 93.98 64.135) (end 92.075 66.04) (width 0.5) (layer F.Cu) (net 19))
+  (segment (start 99.06 64.135) (end 93.98 64.135) (width 0.5) (layer F.Cu) (net 19))
+  (segment (start 103.505 68.58) (end 99.06 64.135) (width 0.5) (layer F.Cu) (net 19))
   (zone (net 1) (net_name GND) (layer B.Cu) (hatch edge 0.508)
     (connect_pads (clearance 0.508))

Commit message: Upgrade to KiCAD 6
Parts:
- moved RV1 5.00 mm to (113.1, 72.4)
Connections:
- J1 pad 2: (no net) -> unconnected-(J1-Pad2)
- RV1 pad 1: +9VA -> unconnected-(RV1-Pad1)
- RV1 pad 3: (no net) -> +9VA
- U2 pad 5: (no net) -> unconnected-(U2-Pad5)
Routing:
- net Clock: track 33.9 -> 32.6 mm
- net Net-(C4-Pad1): track 30.8 -> 30.2 mm
Other:
- net class Default removed
